File: pcb_files/kicad_project/main/Sensores.kicad_sch (KiCad schematic)
At the start: 84 parts

Commit message: Termina ruteo de la rebuild.
Parts:
- S1, S10, S11, S12, S13, S14, S15, S16, S17, S18, S19, S2, S20, S21, S22, S23, S24, S3, S4, S5, S6, S7, S8, S9, SML1, SML2, SMR1, SMR2: value ~ -> (none)
