File: pcb_files/kicad_project/main/main.kicad_sch (KiCad schematic)
At the start: 153 parts, among them IC1 AS5145B-HSST, IC2 AS5145B-HSST, J1 Conn_01x02_Socket, J2 Conn_01x04_Socket, Q1 AON7423, Y1 Crystal_GND24

Commit message: Termina ruteo de la rebuild.
Parts:
- removed CM1, CM11, CM3, CM5, CM7, CM9: 10uF, Capacitor_SMD:C_0402_1005Metric_Pad0.74x0.62mm_HandSolder, symbol Device:C
- removed CM10, CM12, CM2, CM4, CM6, CM8: 0.1uF, Capacitor_SMD:C_0402_1005Metric_Pad0.74x0.62mm_HandSolder, symbol Device:C
- added BTN_MENU1, BTN_MENU2: (no value), custom_footprints:Generic_SmallButton_6x3, symbol custom_symbols:Button
- added CF1, CF2: 0.22uF, Capacitor_SMD:C_0402_1005Metric_Pad0.74x0.62mm_HandSolder, symbol Device:C
- added JPH2, JPH3: JPH2, Jumper:SolderJumper-2_P1.3mm_Open_RoundedPad1.0x1.5mm, symbol Jumper:SolderJumper_2_Open
- added RBTN1, RBTN2: 47k, Resistor_SMD:R_0402_1005Metric_Pad0.72x0.64mm_HandSolder, symbol Device:R
- added RCS1, RCS2, RCS3, RCS4: 5K, Resistor_SMD:R_0402_1005Metric_Pad0.72x0.64mm_HandSolder, symbol Device:R
- added RF1, RF2: 220, Resistor_SMD:R_0402_1005Metric_Pad0.72x0.64mm_HandSolder, symbol Device:R
- BTN_RST1, DC-DC1, IR_RECIVER1, LSM6DSR1, MP1, MP2, USB1: value ~ -> (none)
- CONN_ENC_L1, CONN_ENC_R1: footprint custom_footprints:FujitoraBot2_PCBmodule_encoder -> custom_footprints:DragonBot_PCBmodule_encoder
- ENC_L1, ENC_R1: footprint custom_footprints:DragonBot2_Encoder_main -> custom_footprints:DragonBot2_PCBmain_Encoder
- LDO1: footprint Package_DFN_QFN:DFN-6-1EP_3x3mm_P0.95mm_EP1.7x2.6mm -> custom_footprints:DFN-6-2x2mm_P0.5mm_LDO_Dragonbot
Connections:
- net +3V3: now also BTN_MENU1.1, BTN_MENU2.1, RCS1.1, RCS3.1
- net ENC_L_A: now also DEIXAME_QUE_PENSE_1.57 (PB5); no longer DEIXAME_QUE_PENSE_1.56 (PB4)
- net ENC_L_B: now also DEIXAME_QUE_PENSE_1.56 (PB4); no longer DEIXAME_QUE_PENSE_1.57 (PB5)
- net GND: now also LDO1.7 (PAD), CF1.2, CF2.2, JPH2.2 (B), JPH3.2 (B), RBTN1.2, RBTN2.2, RCS2.1, RCS4.1; no longer MP1.17 (OCMD), MP2.17 (OCMD)
- net IN_CURR_ML_A: no longer names the net of MP1.15 (SOA)
- net IN_CURR_ML_A: now also MP1.16 (SOB), RCS1.2, RCS2.2, RF1.1; no longer DEIXAME_QUE_PENSE_1.20 (PA4)
- net IN_CURR_ML_B renamed CURR_SEN_MR
- net CURR_SEN_MR: now also CF2.1, RF2.2; no longer MP1.16 (SOB)
- net IN_CURR_MR_A: no longer names the net of MP2.15 (SOA)
- net IN_CURR_MR_A: now also MP2.16 (SOB), RCS3.2, RCS4.2, RF2.1; no longer DEIXAME_QUE_PENSE_1.22 (PA6)
- net IN_CURR_MR_B renamed MENU_BTN_R
- net MENU_BTN_R: now also BTN_MENU2.2, RBTN2.1; no longer MP2.16 (SOB)
- net IN_LIN_A renamed IN_MUX_C
- net IN_MUX_C: now also ARRAY_MORRO1.4 (Pin_4); no longer ARRAY_MORRO1.5 (Pin_5)
- net IN_LIN_B renamed IN_MUX_B
- net IN_MUX_B: now also ARRAY_MORRO1.3 (Pin_3); no longer ARRAY_MORRO1.6 (Pin_6)
- net IN_LIN_C renamed IN_MUX_A
- net IN_MUX_A: now also ARRAY_MORRO1.2 (Pin_2); no longer ARRAY_MORRO1.7 (Pin_7)
- net OUT_MUX_A renamed OUT_CH_A
- net OUT_CH_A: now also ARRAY_MORRO1.5 (Pin_5); no longer ARRAY_MORRO1.2 (Pin_2)
- net OUT_MUX_B renamed OUT_CH_B
- net OUT_CH_B: now also ARRAY_MORRO1.6 (Pin_6); no longer ARRAY_MORRO1.3 (Pin_3)
- net OUT_MUX_C renamed OUT_CH_C
- net OUT_CH_C: now also ARRAY_MORRO1.7 (Pin_7); no longer ARRAY_MORRO1.4 (Pin_4)
- new net: JPH2.1 (A), MP2.17 (OCMD)
- new net: JPH3.1 (A), MP1.17 (OCMD)
- new net CURR_SEN_ML: CF1.1, DEIXAME_QUE_PENSE_1.20 (PA4), RF1.2
- new net MENU_BTN_L: BTN_MENU1.2, DEIXAME_QUE_PENSE_1.22 (PA6), RBTN1.1
Other:
- note added: "ACUERDOS: - Morro, PCB flexible blanco - Marcas, PCB flexible blanco - PCB main nueva de 0.8 de color negra con borde blanco. - PCB chasis nueva con nuevos agujeros de grosor... 1mm?"
- note added: "TODO: - Comprobar valores de resistencias de PHs para lectura de corriente (LISTO) - Comprobar que actualmente el mosfet de succion funciona correctamente - Comprobar fuertemente que las conexiones morro PCB estan correctas. (LISTO) - Led encendido izquierdo rootear bien ... MMM no se si se rehara. (NO SE HARA) - Revisar huella de LDO para no poner el LDO de zoro ñapeado (LISTO) - Poner correctam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"
- moved on the sheet: BTN_RST1, BUK9Q20-40H1, CA1, CA2, CDM1, CDM10, CDM2, CDM3, CDM4, CDM5, CDM6, CDM7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
